File: PCB/fusion/BrushlessLamp.sch (EAGLE design)
At the start: 68 parts, among them Q1 PMOS-RevProt

Commit message: PCB: fix reverse-protection FET orientation, Vgs clamp, fuse land + BOM errors
- Q1 P-FET was wired source-to-input: body diode conducted on reversed 24 V
  and the channel blocked nothing. Now drain=input/source=load; gate zener
  clamps G-S and drops 15 V -> 10 V (AO3401A Vgs abs-max is +/-12 V).
- F1: 0466002.NR is a fast NANO2 that didn't fit the 1206 land; now
  0454002.MR slow-blow on a proper NANO2 land (125 V, survives bulk-cap inrush).
- TVS SMBJ30A -> SMBJ28A with honest clamp-margin rationale (full-surge VC
  exceeds the buck's 40 V abs-max; accepted residual risk documented).
- C_BOOT mainboard BOM row said 0.1 uF — the exact value the schematic
  forbids (GPIO0 download-mode strap); now 100 pF C0G.
- BOARD_CUSTOM pin snippet preserves the firmware A/B phase swap (motor spun
  backwards as written); R_AZ encoder pull-up DNP pads now actually exist in
  the netlist (3 added, 71 parts total); R_FBT/R_FBB docs corrected to 0603;
  screw-terminal drills 1.2 -> 1.3 mm; THT count 6 -> 7 (J_EXP); JST-XH 2.50 mm;
  phantom D_OR_5V row removed.
- BrushlessLamp.sch regenerated (71 parts / 57 nets); PCBWay-BOM.xlsx rebuilt
  from the corrected assembly CSV. Verify BZT52C10 / SMBJ28A LCSC numbers and
  the NANO2 land before ordering.

Co-Authored-By: Claude Fable 5 <noreply@anthropic.com>
Parts:
- added R_AZ_A, R_AZ_B, R_AZ_C: 10k-DNP, BLLIB:RES_0603
- D_Q1: value 15V-Zener -> 10V-Zener
- F1: device BLLIB:FUSE_1206 -> BLLIB:FUSE_NANO2
- TVS1: value SMBJ30A -> SMBJ28A
Connections:
- net ENCA: now also R_AZ_A.2
- net ENCB: now also R_AZ_B.2
- net ENCZ: now also R_AZ_C.2
- net P24: now also D_Q1.C, Q1.S; no longer Q1.D
- net P24_F: now also Q1.D; no longer D_Q1.C, Q1.S
- net P3V3: now also R_AZ_A.1, R_AZ_B.1, R_AZ_C.1
Other:
- moved on the sheet: D_CLC, D_CLW, D_USB, J_BTN, J_EXP, J_KNOB, J_LED, J_USB, LED_STATUS, Q_CW, Q_WW, R_GC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
